File: tigard.sch (KiCad schematic (older format))
At the start: 83 parts, among them J1 USB_C_Receptacle_USB2.0, J2 JTAG, J3 UART, J4 SPI, J5 SWD, J6 I2C, Q1 BSH103, SW1 SW_SP3T, SW2 SW_DPDT, SW3 SW_DPDT, U1 AP7365-18, U2 AP7365-33, U3 FT2232HQ, U4 93LC56BT-I/OT, U5 SN74LVC8T245, U6 SN74LVC8T245, Y1 12MHz

Commit message: Re-annotate (fix reference ordering)
Parts:
- renumbered C9 to C10, C10 to C18, C18 to C19, C19 to C20, C20 to C21, C21 to C22, C22 to C9, D5 to D3, D6 to D4, D7 to D5, D3 to D6, D4 to D7, R23 to R10, R24 to R11, R19 to R16, R16 to R17, R17 to R18, R18 to R19, R6 to R20, R7 to R21, R8 to R22, R9 to R23, R10 to R6, R11 to R7, R21 to R8, R22 to R9
Changed lines of the file:
@@
 	9400 3250 9050 3250
 $Comp
-L Device:R_Small R8
+L Device:R_Small R22
 U 1 1 5EC197B6
 P 9500 3300
-F 0 "R8" H 9559 3346 50  0000 L CNN
+F 0 "R22" H 9559 3346 50  0000 L CNN
 F 1 "2.2k" H 9559 3255 50  0000 L CNN
 F 2 "Resistor_SMD:R_0402_1005Metric" H 9500 3300 50  0001 C CNN
@@
 	9050 3550 9750 3550
 $Comp
-L Device:D_Schottky_Small D3
+L Device:D_Schottky_Small D6
 U 1 1 5EC4F33A
 P 10150 3450
-F 0 "D3" H 10150 3243 50  0000 C CNN
+F 0 "D6" H 10150 3243 50  0000 C CNN
 F 1 "RB751S40" H 10150 3334 50  0000 C CNN
 F 2 "Diode_SMD:D_SOD-523" V 10150 3450 50  0001 C CNN
@@
 	10400 3450 10250 3450
 $Comp
-L Device:D_Schottky_Small D4
+L Device:D_Schottky_Small D7
 U 1 1 5EC63806
 P 10150 3550
-F 0 "D4" H 10150 3665 50  0000 C CNN
+F 0 "D7" H 10150 3665 50  0000 C CNN
 F 1 "RB751S40" H 10150 3756 50  0000 C CNN
 F 2 "Diode_SMD:D_SOD-523" V 10150 3550 50  0001 C CNN
@@
 $EndComp
 $Comp
-L Device:R_Small R7
+L Device:R_Small R21
 U 1 1 5EDD63F0
 P 9350 2300
-F 0 "R7" V 9300 2150 50  0000 C CNN
+F 0 "R21" V 9300 2150 50  0000 C CNN
 F 1 "10k" V 9300 2450 50  0000 C CNN
 F 2 "Resistor_SMD:R_0402_1005Metric" H 9350 2300 50  0001 C CNN
@@
 $EndComp
 $Comp
-L Device:R_Small R6
+L Device:R_Small R20
 U 1 1 5EDD6C7C
 P 8350 2400
-F 0 "R6" V 8154 2400 50  0000 C CNN
+F 0 "R20" V 8154 2400 50  0000 C CNN
 F 1 "10k" V 8245 2400 50  0000 C CNN
 F 2 "Resistor_SMD:R_0402_1005Metric" H 8350 2400 50  0001 C CNN
@@
 $EndComp
 $Comp
-L Device:R_Small R9
+L Device:R_Small R23
 U 1 1 5EDDC797
 P 9750 3200
-F 0 "R9" H 9809 3246 50  0000 L CNN
+F 0 "R23" H 9809 3246 50  0000 L CNN
 F 1 "2.2k" H 9809 3155 50  0000 L CNN
 F 2 "Resistor_SMD:R_0402_1005Metric" H 9750 3200 50  0001 C CNN
@@
 VREG
 $Comp
-L Device:C_Small C9
+L Device:C_Small C10
 U 1 1 5EDF954F
 P 1150 4850
-F 0 "C9" H 1242 4896 50  0000 L CNN
+F 0 "C10" H 1242 4896 50  0000 L CNN
 F 1 "2.2u" H 1242 4805 50  0000 L CNN
 F 2 "Capacitor_SMD:C_0603_1608Metric" H 1150 4850 50  0001 C CNN
@@
 USB_DP
 $Comp
-L Device:R_Small R10
+L Device:R_Small R6
 U 1 1 5EE10D01
 P 950 5850
-F 0 "R10" V 754 5850 50  0000 C CNN
+F 0 "R6" V 754 5850 50  0000 C CNN
 F 1 "12k, 1%" V 845 5850 50  0000 C CNN
 F 2 "Resistor_SMD:R_0402_1005Metric" H 950 5850 50  0001 C CNN
@@
 $EndComp
 $Comp
-L Device:R_Small R11
+L Device:R_Small R7
 U 1 1 5EE173E9
 P 1350 6050
-F 0 "R11" V 1246 6050 50  0000 C CNN
+F 0 "R7" V 1246 6050 50  0000 C CNN
 F 1 "10k" V 1155 6050 50  0000 C CNN
 F 2 "Resistor_SMD:R_0402_1005Metric" H 1350 6050 50  0001 C CNN
@@
 	2700 10450 2700 10400
 $Comp
-L Device:C_Small C10
+L Device:C_Small C18
 U 1 1 5F66B1F7
 P 1700 10050
-F 0 "C10" H 1608 10096 50  0000 R CNN
+F 0 "C18" H 1608 10096 50  0000 R CNN
 F 1 "100n" H 1608 10005 50  0000 R CNN
 F 2 "Capacitor_SMD:C_0402_1005Metric" H 1700 10050 50  0001 C CNN
@@
 	5450 6150 5900 6150
 $Comp
-L Device:R_Small R17
+L Device:R_Small R18
 U 1 1 5FB4F232
 P 5600 5200
-F 0 "R17" V 5500 5200 50  0000 C CNN
+F 0 "R18" V 5500 5200 50  0000 C CNN
 F 1 "10k" V 5400 5200 50  0000 C CNN
 F 2 "Resistor_SMD:R_0402_1005Metric" H 5600 5200 50  0001 C CNN
@@
 	5300 7900 5350 7900
 $Comp
-L Device:R_Small R18
+L Device:R_Small R19
 U 1 1 601ADA37
 P 5900 6950
-F 0 "R18" H 5841 6904 50  0000 R CNN
+F 0 "R19" H 5841 6904 50  0000 R CNN
 F 1 "10k" H 5841 6995 50  0000 R CNN
 F 2 "Resistor_SMD:R_0402_1005Metric" H 5900 6950 50  0001 C CNN
@@
 	550  11150 8300 11150
 $Comp
-L Device:C_Small C18
+L Device:C_Small C19
 U 1 1 60D35425
 P 5750 4550
-F 0 "C18" H 5842 4596 50  0000 L CNN
+F 0 "C19" H 5842 4596 50  0000 L CNN
 F 1 "100n" H 5842 4505 50  0000 L CNN
 F 2 "Capacitor_SMD:C_0402_1005Metric" H 5750 4550 50  0001 C CNN
@@
 $EndComp
 $Comp
-L Device:C_Small C19
+L Device:C_Small C20
 U 1 1 60D35DE8
 P 6150 4550
-F 0 "C19" H 6242 4596 50  0000 L CNN
+F 0 "C20" H 6242 4596 50  0000 L CNN
 F 1 "100n" H 6242 4505 50  0000 L CNN
 F 2 "Capacitor_SMD:C_0402_1005Metric" H 6150 4550 50  0001 C CNN
@@
 $EndComp
 $Comp
-L Device:C_Small C20
+L Device:C_Small C21
 U 1 1 60D35F31
 P 6650 4550
-F 0 "C20" H 6742 4596 50  0000 L CNN
+F 0 "C21" H 6742 4596 50  0000 L CNN
 F 1 "100n" H 6742 4505 50  0000 L CNN
 F 2 "Capacitor_SMD:C_0402_1005Metric" H 6650 4550 50  0001 C CNN
@@
 $EndComp
 $Comp
-L Device:C_Small C21
+L Device:C_Small C22
 U 1 1 60D3615E
 P 7050 4550
-F 0 "C21" H 7142 4596 50  0000 L CNN
+F 0 "C22" H 7142 4596 50  0000 L CNN
 F 1 "100n" H 7142 4505 50  0000 L CNN
 F 2 "Capacitor_SMD:C_0402_1005Metric" H 7050 4550 50  0001 C CNN
@@
 VREF
 $Comp
-L Device:R_Small R16
+L Device:R_Small R17
 U 1 1 610CF3DF
 P 7450 4550
-F 0 "R16" H 7509 4596 50  0000 L CNN
+F 0 "R17" H 7509 4596 50  0000 L CNN
 F 1 "1M" H 7509 4505 50  0000 L CNN
 F 2 "Resistor_SMD:R_0402_1005Metric" H 7450 4550 50  0001 C CNN
@@
 	6050 3350 6550 3350
 $Comp
-L Device:R_Small R19
+L Device:R_Small R16
 U 1 1 5EEC3913
 P 7150 3450
-F 0 "R19" V 6954 3450 50  0000 C CNN
+F 0 "R16" V 6954 3450 50  0000 C CNN
 F 1 "330" V 7045 3450 50  0000 C CNN
 F 2 "Resistor_SMD:R_0402_1005Metric" H 7150 3450 50  0001 C CNN
@@
 	4800 4050 11150 4050
 $Comp
-L Device:LED_Small D5
+L Device:LED_Small D3
 U 1 1 5F225D89
 P 4300 5550
-F 0 "D5" V 4346 5647 50  0000 L CNN
+F 0 "D3" V 4346 5647 50  0000 L CNN
 F 1 "GREEN" V 4255 5647 50  0000 L CNN
 F 2 "LED_SMD:LED_0603_1608Metric" V 4300 5550 50  0001 C CNN
@@
 	4250 8150 4450 8150
 $Comp
-L Device:LED_Small D6
+L Device:LED_Small D4
 U 1 1 5FCEB5AF
 P 4450 5550
-F 0 "D6" V 4496 5480 50  0000 R CNN
+F 0 "D4" V 4496 5480 50  0000 R CNN
 F 1 "GREEN" V 4405 5480 50  0000 R CNN
 F 2 "LED_SMD:LED_0603_1608Metric" V 4450 5550 50  0001 C CNN
@@
 $EndComp
 $Comp
-L Device:LED_Small D7
+L Device:LED_Small D5
 U 1 1 5FCEBABB
 P 4450 8000
-F 0 "D7" V 4496 7930 50  0000 R CNN
+F 0 "D5" V 4496 7930 50  0000 R CNN
 F 1 "GREEN" V 4405 7930 50  0000 R CNN
 F 2 "LED_SMD:LED_0603_1608Metric" V 4450 8000 50  0001 C CNN
@@
 $EndComp
 $Comp
-L Device:R_Small R22
+L Device:R_Small R9
 U 1 1 6027FAD3
 P 4450 5300
-F 0 "R22" H 4391 5254 50  0000 R CNN
+F 0 "R9" H 4391 5254 50  0000 R CNN
 F 1 "330" H 4391 5345 50  0000 R CNN
 F 2 "Resistor_SMD:R_0402_1005Metric" H 4450 5300 50  0001 C CNN
@@
 $EndComp
 $Comp
-L Device:R_Small R21
+L Device:R_Small R8
 U 1 1 6027FE9C
 P 4300 5300
-F 0 "R21" H 4358 5254 50  0000 L CNN
+F 0 "R8" H 4358 5254 50  0000 L CNN
 F 1 "330" H 4358 5345 50  0000 L CNN
 F 2 "Resistor_SMD:R_0402_1005Metric" H 4300 5300 50  0001 C CNN
@@
 $EndComp
 $Comp
-L Device:R_Small R24
+L Device:R_Small R11
 U 1 1 60280318
 P 4450 7750
-F 0 "R24" H 4391 7704 50  0000 R CNN
+F 0 "R11" H 4391 7704 50  0000 R CNN
 F 1 "330" H 4391 7795 50  0000 R CNN
 F 2 "Resistor_SMD:R_0402_1005Metric" H 4450 7750 50  0001 C CNN
@@
 $EndComp
 $Comp
-L Device:R_Small R23
+L Device:R_Small R10
 U 1 1 60387B05
 P 4250 7750
-F 0 "R23" H 4192 7796 50  0000 R CNN
+F 0 "R10" H 4192 7796 50  0000 R CNN
 F 1 "10k" H 4192 7705 50  0000 R CNN
 F 2 "Resistor_SMD:R_0402_1005Metric" H 4250 7750 50  0001 C CNN
@@
 $EndComp
 $Comp
-L Device:C_Small C22
+L Device:C_Small C9
 U 1 1 603890D4
 P 950 4850
-F 0 "C22" H 858 4896 50  0000 R CNN
+F 0 "C9" H 858 4896 50  0000 R CNN
 F 1 "2.2u" H 858 4805 50  0000 R CNN
 F 2 "Capacitor_SMD:C_0603_1608Metric" H 950 4850 50  0001 C CNN
